Commit message: Mesh paths are now relative

File: src/hunav_gazebo_wrapper-humble/media/models/ceres_alpha.urdf (robot description, URDF)
Before this commit: robot ceres_alpha, 7 links, 6 joints
Links:
- link base_link: geometry collision mesh filename=/meshes/base_link.STL; visual mesh filename=/meshes/base_link.STL
- link caster_left_link_1: geometry collision mesh filename=/meshes/caster_left_link_1.STL; visual mesh filename=/meshes/caster_left_link_1.STL
- link caster_right_link_1: geometry collision mesh filename=/meshes/caster_right_link_1.STL; visual mesh filename=/meshes/caster_right_link_1.STL
- link caster_wheel_left_link_1: geometry collision mesh filename=/meshes/caster_wheel_left_link_1.STL; visual mesh filename=/meshes/caster_wheel_left_link_1.STL
- link caster_wheel_right_link_1: geometry collision mesh filename=/meshes/caster_wheel_right_link_1.STL; visual mesh filename=/meshes/caster_wheel_right_link_1.STL
- link left_drive_wheel_link_1: geometry collision mesh filename=/meshes/left_drive_wheel_link_1.STL; visual mesh filename=/meshes/left_drive_wheel_link_1.STL
- link right_drive_wheel_link_1: geometry collision mesh filename=/meshes/right_drive_wheel_link_1.STL; visual mesh filename=/meshes/right_drive_wheel_link_1.STL

Commit message: Using standard joystick package

File: src/hunav_gazebo_wrapper-humble/media/models/ceres_alpha.urdf (robot description, URDF)
Before this commit: robot ceres_alpha, 7 links, 6 joints
Links:
- link base_link: mass 37.2854108654229 -> 18.2854108654229

Commit message: Add lidar to alpha ceres

File: src/hunav_gazebo_wrapper-humble/media/models/ceres_alpha.urdf (robot description, URDF)
Before this commit: robot ceres_alpha, 7 links, 6 joints
Links:
- added link laser_frame; collision cylinder length=0.02 radius=0.025; visual cylinder length=0.02 radius=0.025
Joints:
- added joint laser_joint: type fixed, parent base_link, child laser_frame, origin xyz=-0.39 0 -0.05 rpy=0 0 0

Commit message: nav2 (WIP)

File: src/hunav_gazebo_wrapper-humble/media/models/ceres_alpha.urdf (robot description, URDF)
Before this commit: robot ceres_alpha, 8 links, 7 joints
Links:
- link base_link: mass 18.2854108654229 -> 2.2854108654229

Commit message: Fix position of lidar
Swap lidar to front since we're actually driving forwards now.

File: src/hunav_gazebo_wrapper-humble/media/models/ceres_alpha.urdf (robot description, URDF)
Before this commit: robot ceres_alpha, 8 links, 7 joints
Joints:
- joint laser_joint: origin xyz=-0.39 0 -0.05 rpy=0 0 0 -> xyz=0.57 0 -0.06 rpy=0 0 3.145

Commit message: Move lidar to bottom of robot

File: src/hunav_gazebo_wrapper-humble/media/models/ceres_alpha.urdf (robot description, URDF)
Before this commit: robot ceres_alpha, 8 links, 7 joints
Joints:
- joint laser_joint: origin xyz=0.57 0 -0.06 rpy=0 0 3.145 -> xyz=0.57 0 -0.4 rpy=0 0 3.145

Commit message: Move lidar to middle

File: src/hunav_gazebo_wrapper-humble/media/models/ceres_alpha.urdf (robot description, URDF)
Before this commit: robot ceres_alpha, 8 links, 7 joints
Joints:
- joint laser_joint: origin xyz=0.57 0 -0.4 rpy=0 0 3.145 -> xyz=0.15 0 -0.4 rpy=0 0 3.145
