Commit message: Move Alpha Ceres urdf

File: src/validate/models/ceres_alpha.urdf (robot description, URDF)
Before this commit: robot ceres_alpha, 8 links, 7 joints
Links:
- added link base_footprint
Joints:
- added joint base_joint: type fixed, parent base_footprint, child base_link, origin xyz=0 0 0.825 rpy=0 0 0
